File: RotaryEncoderBreakout.sch (KiCad schematic (older format))
At the start: 18 parts, among them J1 Conn_01x04_Male, J2 Conn_01x04_Male, J3 Conn_01x03_Male, SW1 RotaryEncoder_Switch_RGB, U1 WS2811

Commit message: Layout complete
Parts:
- removed J3: Conn_01x03_Male, Pin_Headers:Pin_Header_Straight_1x03_Pitch2.54mm, symbol Conn_01x03_Male
- removed R9: 0R, Resistors_SMD:R_0805_HandSoldering, symbol R
- added J3: Conn_01x05_Male, Pin_Headers:Pin_Header_Straight_1x05_Pitch2.54mm, symbol Conn_01x05_Male
Connections:
- net +5V: now also J2.4 (Pin_4), J3.5 (Pin_5); no longer J2.1 (Pin_1)
- net at U1.5 (DOUT): now also J3.3 (Pin_3)
- net at U1.7 (SET): now also J3.4 (Pin_4)
- net at C1.1, R2.2: now also J1.3 (Pin_3); no longer J1.2 (Pin_2)
- net at C2.1, R3.2: now also J1.2 (Pin_2); no longer J1.3 (Pin_3)
- net at C4.1, R8.2: now also J1.4 (Pin_4); no longer J1.1 (Pin_1)
- net at R7.2: now also J3.2 (Pin_2)
- new net: J1.1 (Pin_1), J3.1 (Pin_1)
Changed lines of the file:
@@
 L Conn_01x04_Male J2
 U 1 1 5A22155E
-P 3700 2750
-F 0 "J2" H 3700 2950 50  0000 C CNN
-F 1 "Conn_01x04_Male" H 3700 2450 50  0000 C CNN
-F 2 "Pin_Headers:Pin_Header_Angled_1x04_Pitch2.54mm" H 3700 2750 50  0001 C CNN
-F 3 "" H 3700 2750 50  0001 C CNN
-	1    3700 2750
-	1    0    0    -1
+P 3700 2850
+F 0 "J2" H 3700 3050 50  0000 C CNN
+F 1 "Conn_01x04_Male" H 3700 2550 50  0000 C CNN
+F 2 "Pin_Headers:Pin_Header_Angled_1x04_Pitch2.54mm" H 3700 2850 50  0001 C CNN
+F 3 "" H 3700 2850 50  0001 C CNN
+	1    3700 2850
+	1    0    0    1
 $EndComp
 $Comp
@@
 L Conn_01x04_Male J1
 U 1 1 5A222349
-P 3700 3450
-F 0 "J1" H 3700 3650 50  0000 C CNN
-F 1 "Conn_01x04_Male" H 3700 3150 50  0000 C CNN
-F 2 "Pin_Headers:Pin_Header_Angled_1x04_Pitch2.54mm" H 3700 3450 50  0001 C CNN
-F 3 "" H 3700 3450 50  0001 C CNN
-	1    3700 3450
-	1    0    0    -1
+P 3700 3550
+F 0 "J1" H 3700 3750 50  0000 C CNN
+F 1 "Conn_01x04_Male" H 3700 3250 50  0000 C CNN
+F 2 "Pin_Headers:Pin_Header_Angled_1x04_Pitch2.54mm" H 3700 3550 50  0001 C CNN
+F 3 "" H 3700 3550 50  0001 C CNN
+	1    3700 3550
+	1    0    0    1
 $EndComp
 Text Label 3550 3650 2    60   ~ 0
@@
 	4000 3650 4000 4650
 Wire Wire Line
-	4000 4650 9350 4650
+	4000 4650 8900 4650
 Wire Wire Line
 	6900 3400 7050 3400
@@
 $EndComp
 Wire Wire Line
-	9350 4650 9350 2950
+	8900 4650 8900 3350
 $Comp
 L C C4
@@
 	6600 4000 7050 4000
 Connection ~ 7050 4000
-$Comp
-L Conn_01x03_Male J3
-U 1 1 5A2603E6
-P 9100 3250
-F 0 "J3" H 9100 3450 50  0000 C CNN
-F 1 "Conn_01x03_Male" H 9100 3050 50  0000 C CNN
-F 2 "Pin_Headers:Pin_Header_Straight_1x03_Pitch2.54mm" H 9100 3250 50  0001 C CNN
-F 3 "" H 9100 3250 50  0001 C CNN
-	1    9100 3250
-	-1   0    0    1
-$EndComp
-Wire Wire Line
-	9350 2950 8900 2950
-Wire Wire Line
-	8900 2950 8900 3150
 Wire Wire Line
 	8800 3250 8900 3250
@@
 	8400 3250 8500 3250
 Wire Wire Line
-	8400 3350 8900 3350
-$Comp
-L R R9
-U 1 1 5A260AC7
-P 8550 2850
-F 0 "R9" V 8630 2850 50  0000 C CNN
-F 1 "0R" V 8550 2850 50  0000 C CNN
-F 2 "Resistors_SMD:R_0805_HandSoldering" V 8480 2850 50  0001 C CNN
-F 3 "" H 8550 2850 50  0001 C CNN
-	1    8550 2850
-	1    0    0    -1
-$EndComp
-Wire Wire Line
 	8400 3150 8550 3150
 Wire Wire Line
-	8550 3150 8550 3000
+	8550 3150 8550 3050
 $Comp
 L +5V #PWR018
 U 1 1 5A260D0D
-P 8550 2600
-F 0 "#PWR018" H 8550 2450 50  0001 C CNN
-F 1 "+5V" H 8550 2740 50  0000 C CNN
-F 2 "" H 8550 2600 50  0001 C CNN
-F 3 "" H 8550 2600 50  0001 C CNN
-	1    8550 2600
-	1    0    0    -1
-$EndComp
-Wire Wire Line
-	8550 2600 8550 2700
+P 8750 2900
+F 0 "#PWR018" H 8750 2750 50  0001 C CNN
+F 1 "+5V" H 8750 3040 50  0000 C CNN
+F 2 "" H 8750 2900 50  0001 C CNN
+F 3 "" H 8750 2900 50  0001 C CNN
+	1    8750 2900
+	1    0    0    -1
+$EndComp
+$Comp
+L Conn_01x05_Male J3
+U 1 1 5A28BDF7
+P 9100 3150
+F 0 "J3" H 9100 3450 50  0000 C CNN
+F 1 "Conn_01x05_Male" V 8900 3150 50  0000 C CNN
+F 2 "Pin_Headers:Pin_Header_Straight_1x05_Pitch2.54mm" H 9100 3150 50  0001 C CNN
+F 3 "" H 9100 3150 50  0001 C CNN
+	1    9100 3150
+	-1   0    0    1
+$EndComp
+Wire Wire Line
+	8550 3050 8900 3050
+Wire Wire Line
+	8750 2900 8750 2950
+Wire Wire Line
+	8750 2950 8900 2950
+Wire Wire Line
+	8400 3350 8850 3350
+Wire Wire Line
+	8850 3350 8850 3150
+Wire Wire Line
+	8850 3150 8900 3150
 $EndSCHEMATC

Commit message: Changed symbol and library references to local copy
Parts:
- C1, C2, C3, C4: footprint Capacitors_SMD:C_0805_HandSoldering -> lib_fp:C_0805_HandSoldering
- J1, J2: footprint Pin_Headers:Pin_Header_Angled_1x04_Pitch2.54mm -> lib_fp:Pin_Header_Straight_1x04_Pitch2.54mm
- J3: footprint Pin_Headers:Pin_Header_Straight_1x05_Pitch2.54mm -> lib_fp:Pin_Header_Straight_1x05_Pitch2.54mm
- R1, R2, R3, R4, R5, R6, R7, R8: footprint Resistors_SMD:R_0805_HandSoldering -> lib_fp:R_0805_HandSoldering
- U1: footprint Housings_SOIC:SOIC-8_3.9x4.9mm_Pitch1.27mm -> lib_fp:SOIC-8_3.9x4.9mm_Pitch1.27mm
Changed lines of the file:
@@
 EESchema Schematic File Version 2
+LIBS:RotaryEncoderBreakout
 LIBS:power
 LIBS:device
@@
 F 0 "U1" H 7725 3150 60  0000 C CNN
 F 1 "WS2811" H 7650 3625 60  0000 C CNN
-F 2 "Housings_SOIC:SOIC-8_3.9x4.9mm_Pitch1.27mm" H 7900 3300 60  0001 C CNN
+F 2 "lib_fp:SOIC-8_3.9x4.9mm_Pitch1.27mm" H 7900 3300 60  0001 C CNN
 F 3 "" H 7900 3300 60  0001 C CNN
 	1    7900 3300
@@
 F 0 "J2" H 3700 3050 50  0000 C CNN
 F 1 "Conn_01x04_Male" H 3700 2550 50  0000 C CNN
-F 2 "Pin_Headers:Pin_Header_Angled_1x04_Pitch2.54mm" H 3700 2850 50  0001 C CNN
+F 2 "lib_fp:Pin_Header_Straight_1x04_Pitch2.54mm" H 3700 2850 50  0001 C CNN
 F 3 "" H 3700 2850 50  0001 C CNN
 	1    3700 2850
@@
 F 0 "R5" V 5480 2850 50  0000 C CNN
 F 1 "10K" V 5400 2850 50  0000 C CNN
-F 2 "Resistors_SMD:R_0805_HandSoldering" V 5330 2850 50  0001 C CNN
+F 2 "lib_fp:R_0805_HandSoldering" V 5330 2850 50  0001 C CNN
 F 3 "" H 5400 2850 50  0001 C CNN
 	1    5400 2850
@@
 F 0 "R2" V 4930 3200 50  0000 C CNN
 F 1 "10K" V 4850 3200 50  0000 C CNN
-F 2 "Resistors_SMD:R_0805_HandSoldering" V 4780 3200 50  0001 C CNN
+F 2 "lib_fp:R_0805_HandSoldering" V 4780 3200 50  0001 C CNN
 F 3 "" H 4850 3200 50  0001 C CNN
 	1    4850 3200
@@
 F 0 "C1" H 4625 3500 50  0000 L CNN
 F 1 ".01uF" H 4625 3300 50  0000 L CNN
-F 2 "Capacitors_SMD:C_0805_HandSoldering" H 4638 3250 50  0001 C CNN
+F 2 "lib_fp:C_0805_HandSoldering" H 4638 3250 50  0001 C CNN
 F 3 "" H 4600 3400 50  0001 C CNN
 	1    4600 3400
@@
 F 0 "C2" H 4625 4100 50  0000 L CNN
 F 1 ".01uF" H 4625 3900 50  0000 L CNN
-F 2 "Capacitors_SMD:C_0805_HandSoldering" H 4638 3850 50  0001 C CNN
+F 2 "lib_fp:C_0805_HandSoldering" H 4638 3850 50  0001 C CNN
 F 3 "" H 4600 4000 50  0001 C CNN
 	1    4600 4000
@@
 F 0 "R3" V 4930 3800 50  0000 C CNN
 F 1 "10K" V 4850 3800 50  0000 C CNN
-F 2 "Resistors_SMD:R_0805_HandSoldering" V 4780 3800 50  0001 C CNN
+F 2 "lib_fp:R_0805_HandSoldering" V 4780 3800 50  0001 C CNN
 F 3 "" H 4850 3800 50  0001 C CNN
 	1    4850 3800
@@
 F 0 "R4" V 5180 2850 50  0000 C CNN
 F 1 "10K" V 5100 2850 50  0000 C CNN
-F 2 "Resistors_SMD:R_0805_HandSoldering" V 5030 2850 50  0001 C CNN
+F 2 "lib_fp:R_0805_HandSoldering" V 5030 2850 50  0001 C CNN
 F 3 "" H 5100 2850 50  0001 C CNN
 	1    5100 2850
@@
 F 0 "J1" H 3700 3750 50  0000 C CNN
 F 1 "Conn_01x04_Male" H 3700 3250 50  0000 C CNN
-F 2 "Pin_Headers:Pin_Header_Angled_1x04_Pitch2.54mm" H 3700 3550 50  0001 C CNN
+F 2 "lib_fp:Pin_Header_Straight_1x04_Pitch2.54mm" H 3700 3550 50  0001 C CNN
 F 3 "" H 3700 3550 50  0001 C CNN
 	1    3700 3550
@@
 F 0 "R1" V 7130 4200 50  0000 C CNN
 F 1 "10K" V 7050 4200 50  0000 C CNN
-F 2 "Resistors_SMD:R_0805_HandSoldering" V 6980 4200 50  0001 C CNN
+F 2 "lib_fp:R_0805_HandSoldering" V 6980 4200 50  0001 C CNN
 F 3 "" H 7050 4200 50  0001 C CNN
 	1    7050 4200
@@
 F 0 "R6" V 7980 2500 50  0000 C CNN
 F 1 "100" V 7900 2500 50  0000 C CNN
-F 2 "Resistors_SMD:R_0805_HandSoldering" V 7830 2500 50  0001 C CNN
+F 2 "lib_fp:R_0805_HandSoldering" V 7830 2500 50  0001 C CNN
 F 3 "" H 7900 2500 50  0001 C CNN
 	1    7900 2500
@@
 F 0 "C3" H 8125 2850 50  0000 L CNN
 F 1 ".1uF" H 8125 2650 50  0000 L CNN
-F 2 "Capacitors_SMD:C_0805_HandSoldering" H 8138 2600 50  0001 C CNN
+F 2 "lib_fp:C_0805_HandSoldering" H 8138 2600 50  0001 C CNN
 F 3 "" H 8100 2750 50  0001 C CNN
 	1    8100 2750
@@
 F 0 "R7" V 8730 3250 50  0000 C CNN
 F 1 "33" V 8650 3250 50  0000 C CNN
-F 2 "Resistors_SMD:R_0805_HandSoldering" V 8580 3250 50  0001 C CNN
+F 2 "lib_fp:R_0805_HandSoldering" V 8580 3250 50  0001 C CNN
 F 3 "" H 8650 3250 50  0001 C CNN
 	1    8650 3250
@@
 F 0 "C4" H 6225 4300 50  0000 L CNN
 F 1 ".01uF" H 6225 4100 50  0000 L CNN
-F 2 "Capacitors_SMD:C_0805_HandSoldering" H 6238 4050 50  0001 C CNN
+F 2 "lib_fp:C_0805_HandSoldering" H 6238 4050 50  0001 C CNN
 F 3 "" H 6200 4200 50  0001 C CNN
 	1    6200 4200
@@
 F 0 "R8" V 6530 4000 50  0000 C CNN
 F 1 "10K" V 6450 4000 50  0000 C CNN
-F 2 "Resistors_SMD:R_0805_HandSoldering" V 6380 4000 50  0001 C CNN
+F 2 "lib_fp:R_0805_HandSoldering" V 6380 4000 50  0001 C CNN
 F 3 "" H 6450 4000 50  0001 C CNN
 	1    6450 4000
@@
 F 0 "J3" H 9100 3450 50  0000 C CNN
 F 1 "Conn_01x05_Male" V 8900 3150 50  0000 C CNN
-F 2 "Pin_Headers:Pin_Header_Straight_1x05_Pitch2.54mm" H 9100 3150 50  0001 C CNN
+F 2 "lib_fp:Pin_Header_Straight_1x05_Pitch2.54mm" H 9100 3150 50  0001 C CNN
 F 3 "" H 9100 3150 50  0001 C CNN
 	1    9100 3150
