File: RotaryEncoderBreakout.sch (KiCad schematic (older format))
At the start: 17 parts, among them J1 Conn_01x04_Male, J2 Conn_01x04_Male, J3 Conn_01x05_Male, SW1 RotaryEncoder_Switch_RGB, U1 WS2811

Commit message: Update component values
Parts:
- C1, C2, C4: value .01uF -> .1uF
- R2, R3, R8: value 10K -> 22K
Changed lines of the file:
@@
 P 4200 3700
 F 0 "R2" V 4280 3700 50  0000 C CNN
-F 1 "10K" V 4200 3700 50  0000 C CNN
+F 1 "22K" V 4200 3700 50  0000 C CNN
 F 2 "lib_fp:R_0805_HandSoldering" V 4130 3700 50  0001 C CNN
 F 3 "" H 4200 3700 50  0001 C CNN
@@
 P 3950 3900
 F 0 "C1" H 3975 4000 50  0000 L CNN
-F 1 ".01uF" H 3975 3800 50  0000 L CNN
+F 1 ".1uF" H 3975 3800 50  0000 L CNN
 F 2 "lib_fp:C_0805_HandSoldering" H 3988 3750 50  0001 C CNN
 F 3 "" H 3950 3900 50  0001 C CNN
@@
 P 3950 4500
 F 0 "C2" H 3975 4600 50  0000 L CNN
-F 1 ".01uF" H 3975 4400 50  0000 L CNN
+F 1 ".1uF" H 3975 4400 50  0000 L CNN
 F 2 "lib_fp:C_0805_HandSoldering" H 3988 4350 50  0001 C CNN
 F 3 "" H 3950 4500 50  0001 C CNN
@@
 P 4200 4300
 F 0 "R3" V 4280 4300 50  0000 C CNN
-F 1 "10K" V 4200 4300 50  0000 C CNN
+F 1 "22K" V 4200 4300 50  0000 C CNN
 F 2 "lib_fp:R_0805_HandSoldering" V 4130 4300 50  0001 C CNN
 F 3 "" H 4200 4300 50  0001 C CNN
@@
 P 5550 4700
 F 0 "C4" H 5575 4800 50  0000 L CNN
-F 1 ".01uF" H 5575 4600 50  0000 L CNN
+F 1 ".1uF" H 5575 4600 50  0000 L CNN
 F 2 "lib_fp:C_0805_HandSoldering" H 5588 4550 50  0001 C CNN
 F 3 "" H 5550 4700 50  0001 C CNN
@@
 P 5800 4500
 F 0 "R8" V 5880 4500 50  0000 C CNN
-F 1 "10K" V 5800 4500 50  0000 C CNN
+F 1 "22K" V 5800 4500 50  0000 C CNN
 F 2 "lib_fp:R_0805_HandSoldering" V 5730 4500 50  0001 C CNN
 F 3 "" H 5800 4500 50  0001 C CNN
