File: kicad/RotaryEncoderBreakout.sch (KiCad schematic (older format))
At the start: 17 parts, among them J1 Conn_01x04_Male, J2 Conn_01x04_Male, J3 Conn_01x05_Male, SW1 EC12PLRGB, U1 WS2811

Commit message: Add bill of materials
Parts:
- C1, C2, C3, C4: Dist. Part No. (none) -> C0805C104M5RACTU; Dist. URL (none) -> https://www.mouser.com/ProductDetail/80-C0805C104M5R; Distributor (none) -> Mouser
- R1: Dist. Part No. (none) -> 603-RC0805FR-0710KL; Dist. URL (none) -> https://www.mouser.com/ProductDetail/603-RC0805FR-0710KL; Distributor (none) -> Mouser
- R2, R3, R8: Dist. Part No. (none) -> RC0805FR-0722KL; Dist. URL (none) -> https://www.mouser.com/ProductDetail/603-RC0805FR-0722KL; Distributor (none) -> Mouser
- R4, R5: Dist. Part No. (none) -> RC0805FR-0710KL; Dist. URL (none) -> https://www.mouser.com/ProductDetail/603-RC0805FR-0710KL; Distributor (none) -> Mouser
- R6: Dist. Part No. (none) -> 603-RC0805FR-07100RL; Dist. URL (none) -> https://www.mouser.com/ProductDetail/603-RC0805FR-07100RL; Distributor (none) -> Mouser
- R7: Dist. Part No. (none) -> RC0805FR-0733RL; Dist. URL (none) -> https://www.mouser.com/ProductDetail/603-RC0805FR-0733RL; Distributor (none) -> Mouser
- SW1: Dist. Part No. (none) -> 10982; Dist. URL (none) -> https://www.sparkfun.com/products/10982; Distributor (none) -> SparkFun
- U1: Dist. Part No. (none) -> 485-1378; Dist. URL (none) -> https://www.mouser.com/ProductDetail/Adafruit/1378/?qs=%2fh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; Distributor (none) -> Mouser
Changed lines of the file:
@@
 F 2 "lib_fp:SOIC-8_3.9x4.9mm_Pitch1.27mm" H 7250 3800 60  0001 C CNN
 F 3 "" H 7250 3800 60  0001 C CNN
+F 4 "Mouser" H 7250 3800 60  0001 C CNN "Distributor"
+F 5 "485-1378" H 7250 3800 60  0001 C CNN "Dist. Part No."
+F 6 "https://www.mouser.com/ProductDetail/Adafruit/1378/?qs=%2fha2pyFadujIsUxzuHfqvCEPPtKxbz3Fteyuvyy64JU%3d" H 7250 3800 60  0001 C CNN "Dist. URL"
 	1    7250 3800
 	1    0    0    -1
@@
 F 2 "lib_fp:R_0805_HandSoldering" V 4680 3350 50  0001 C CNN
 F 3 "" H 4750 3350 50  0001 C CNN
+F 4 "Mouser" H 4750 3350 60  0001 C CNN "Distributor"
+F 5 "RC0805FR-0710KL" H 4750 3350 60  0001 C CNN "Dist. Part No."
+F 6 "https://www.mouser.com/ProductDetail/603-RC0805FR-0710KL" H 4750 3350 60  0001 C CNN "Dist. URL"
 	1    4750 3350
 	1    0    0    -1
@@
 F 2 "lib_fp:R_0805_HandSoldering" V 4130 3700 50  0001 C CNN
 F 3 "" H 4200 3700 50  0001 C CNN
+F 4 "Mouser" H 4200 3700 60  0001 C CNN "Distributor"
+F 5 "RC0805FR-0722KL" H 4200 3700 60  0001 C CNN "Dist. Part No."
+F 6 "https://www.mouser.com/ProductDetail/603-RC0805FR-0722KL" H 4200 3700 60  0001 C CNN "Dist. URL"
 	1    4200 3700
 	0    1    1    0
@@
 F 2 "lib_fp:C_0805_HandSoldering" H 3988 3750 50  0001 C CNN
 F 3 "" H 3950 3900 50  0001 C CNN
+F 4 "Mouser" H 3950 3900 60  0001 C CNN "Distributor"
+F 5 "C0805C104M5RACTU" H 3950 3900 60  0001 C CNN "Dist. Part No."
+F 6 "https://www.mouser.com/ProductDetail/80-C0805C104M5R" H 3950 3900 60  0001 C CNN "Dist. URL"
 	1    3950 3900
 	1    0    0    -1
@@
 F 2 "lib_fp:C_0805_HandSoldering" H 3988 4350 50  0001 C CNN
 F 3 "" H 3950 4500 50  0001 C CNN
+F 4 "Mouser" H 3950 4500 60  0001 C CNN "Distributor"
+F 5 "C0805C104M5RACTU" H 3950 4500 60  0001 C CNN "Dist. Part No."
+F 6 "https://www.mouser.com/ProductDetail/80-C0805C104M5R" H 3950 4500 60  0001 C CNN "Dist. URL"
 	1    3950 4500
 	1    0    0    -1
@@
 F 2 "lib_fp:R_0805_HandSoldering" V 4130 4300 50  0001 C CNN
 F 3 "" H 4200 4300 50  0001 C CNN
+F 4 "Mouser" H 4200 4300 60  0001 C CNN "Distributor"
+F 5 "RC0805FR-0722KL" H 4200 4300 60  0001 C CNN "Dist. Part No."
+F 6 "https://www.mouser.com/ProductDetail/603-RC0805FR-0722KL" H 4200 4300 60  0001 C CNN "Dist. URL"
 	1    4200 4300
 	0    1    1    0
@@
 F 2 "lib_fp:R_0805_HandSoldering" V 4380 3350 50  0001 C CNN
 F 3 "" H 4450 3350 50  0001 C CNN
+F 4 "Mouser" H 4450 3350 60  0001 C CNN "Distributor"
+F 5 "RC0805FR-0710KL" H 4450 3350 60  0001 C CNN "Dist. Part No."
+F 6 "https://www.mouser.com/ProductDetail/603-RC0805FR-0710KL" H 4450 3350 60  0001 C CNN "Dist. URL"
 	1    4450 3350
 	1    0    0    -1
@@
 F 2 "lib_fp:R_0805_HandSoldering" V 6330 4700 50  0001 C CNN
 F 3 "" H 6400 4700 50  0001 C CNN
+F 4 "Mouser" H 6400 4700 60  0001 C CNN "Distributor"
+F 5 "603-RC0805FR-0710KL" H 6400 4700 60  0001 C CNN "Dist. Part No."
+F 6 "https://www.mouser.com/ProductDetail/603-RC0805FR-0710KL" H 6400 4700 60  0001 C CNN "Dist. URL"
 	1    6400 4700
 	1    0    0    -1
@@
 F 2 "lib_fp:R_0805_HandSoldering" V 7180 3000 50  0001 C CNN
 F 3 "" H 7250 3000 50  0001 C CNN
+F 4 "Mouser" H 7250 3000 60  0001 C CNN "Distributor"
+F 5 "603-RC0805FR-07100RL" H 7250 3000 60  0001 C CNN "Dist. Part No."
+F 6 "https://www.mouser.com/ProductDetail/603-RC0805FR-07100RL" H 7250 3000 60  0001 C CNN "Dist. URL"
 	1    7250 3000
 	1    0    0    -1
@@
 F 2 "lib_fp:C_0805_HandSoldering" H 7488 3100 50  0001 C CNN
 F 3 "" H 7450 3250 50  0001 C CNN
+F 4 "Mouser" H 7450 3250 60  0001 C CNN "Distributor"
+F 5 "C0805C104M5RACTU" H 7450 3250 60  0001 C CNN "Dist. Part No."
+F 6 "https://www.mouser.com/ProductDetail/80-C0805C104M5R" H 7450 3250 60  0001 C CNN "Dist. URL"
 	1    7450 3250
 	0    1    1    0
@@
 F 2 "lib_fp:R_0805_HandSoldering" V 7930 3750 50  0001 C CNN
 F 3 "" H 8000 3750 50  0001 C CNN
+F 4 "Mouser" H 8000 3750 60  0001 C CNN "Distributor"
+F 5 "RC0805FR-0733RL" H 8000 3750 60  0001 C CNN "Dist. Part No."
+F 6 "https://www.mouser.com/ProductDetail/603-RC0805FR-0733RL" H 8000 3750 60  0001 C CNN "Dist. URL"
 	1    8000 3750
 	0    -1   -1   0
@@
 F 2 "lib_fp:C_0805_HandSoldering" H 5588 4550 50  0001 C CNN
 F 3 "" H 5550 4700 50  0001 C CNN
+F 4 "Mouser" H 5550 4700 60  0001 C CNN "Distributor"
+F 5 "C0805C104M5RACTU" H 5550 4700 60  0001 C CNN "Dist. Part No."
+F 6 "https://www.mouser.com/ProductDetail/80-C0805C104M5R" H 5550 4700 60  0001 C CNN "Dist. URL"
 	1    5550 4700
 	1    0    0    -1
@@
 F 2 "lib_fp:R_0805_HandSoldering" V 5730 4500 50  0001 C CNN
 F 3 "" H 5800 4500 50  0001 C CNN
+F 4 "Mouser" H 5800 4500 60  0001 C CNN "Distributor"
+F 5 "RC0805FR-0722KL" H 5800 4500 60  0001 C CNN "Dist. Part No."
+F 6 "https://www.mouser.com/ProductDetail/603-RC0805FR-0722KL" H 5800 4500 60  0001 C CNN "Dist. URL"
 	1    5800 4500
 	0    1    1    0
@@
 F 2 "" H 5550 3825 60  0001 C CNN
 F 3 "" H 5550 3825 60  0001 C CNN
+F 4 "SparkFun" H 5550 3900 60  0001 C CNN "Distributor"
+F 5 "10982" H 5550 3900 60  0001 C CNN "Dist. Part No."
+F 6 "https://www.sparkfun.com/products/10982" H 5550 3900 60  0001 C CNN "Dist. URL"
 	1    5550 3900
 	0    1    1    0

Commit message: Change J1 and J2 to socket headers
Change J1 & J2 from pin headers to Arduino-style socket strips.
Parts:
- J1, J2: footprint lib_fp:Pin_Header_Straight_1x04_Pitch2.54mm -> lib_fp:Socket_Strip_Straight_1x04_Pitch2.54mm
- SW1: footprint (none) -> lib_fp:EC12PLRGB_Rotary_Encoder
Changed lines of the file:
@@
 F 0 "J2" H 3050 3550 50  0000 C CNN
 F 1 "Conn_01x04_Male" H 3050 3050 50  0000 C CNN
-F 2 "lib_fp:Pin_Header_Straight_1x04_Pitch2.54mm" H 3050 3350 50  0001 C CNN
+F 2 "lib_fp:Socket_Strip_Straight_1x04_Pitch2.54mm" H 3050 3350 50  0001 C CNN
 F 3 "" H 3050 3350 50  0001 C CNN
 	1    3050 3350
@@
 F 0 "J1" H 3050 4250 50  0000 C CNN
 F 1 "Conn_01x04_Male" H 3050 3750 50  0000 C CNN
-F 2 "lib_fp:Pin_Header_Straight_1x04_Pitch2.54mm" H 3050 4050 50  0001 C CNN
+F 2 "lib_fp:Socket_Strip_Straight_1x04_Pitch2.54mm" H 3050 4050 50  0001 C CNN
 F 3 "" H 3050 4050 50  0001 C CNN
 	1    3050 4050
@@
 F 0 "SW1" V 5900 3900 60  0000 C CNN
 F 1 "EC12PLRGB" V 5050 3750 40  0000 C CNN
-F 2 "" H 5550 3825 60  0001 C CNN
+F 2 "lib_fp:EC12PLRGB_Rotary_Encoder" H 5550 3825 60  0001 C CNN
 F 3 "" H 5550 3825 60  0001 C CNN
 F 4 "SparkFun" H 5550 3900 60  0001 C CNN "Distributor"
